Commit message: Updated states

File: v2scara/src/description/robot.urdf.xacro (robot description, xacro)
@@ -3,5 +3,5 @@
     <link name="world"></link>
     <joint name="base_joint" type="fixed">
-        <origin xyz="0 0 0" rpy="0 0 0"/>
+        <origin xyz="1 1 0" rpy="0 0 0"/>
         <parent link="world"/>
         <child link="base_link"/>
@@ -9,7 +9,7 @@
     <link name="base_link">
         <visual>
-            <origin xyz="0 0.25 0" rpy="0 0 0"/>
+            <origin xyz="0 0 0.2225" rpy="0 0 0"/>
             <geometry>
-                <box size="0.1 0.5 0.1" />
+                <box size="0.1 0.062 0.445" />
             </geometry>
             <material name="green">
@@ -17,10 +17,27 @@
             </material>
         </visual>
-        <collision>
+        <inertial>
             <origin xyz="0 0 0" rpy="0 0 0"/>
+            <mass value="12" />
+            <inertia ixx="2.26" ixy="0.0" ixz="0.0" iyy="6.26" iyz="0.0" izz="8.5" />
+        </inertial>
+    </link>
+    <joint name="slider_joint" type="prismatic">
+        <origin xyz="0 0 0.445" rpy="0 0 0"/>
+        <parent link="base_link"/>
+        <child link="slider_link"/>
+        <axis xyz="0 0 1"/>
+        <limit lower="-0.445" upper="0" velocity="100" effort="100"/>
+    </joint>
+    <link name="slider_link">
+        <visual>
+            <origin xyz="0 0.049 0" rpy="0 0 0"/>
             <geometry>
-                <box size="2.5 1.5 0.1" />
+                <box size="0.062 0.039 0.052" />
             </geometry>
-        </collision>
+            <material name="green">
+                <color rgba="0.2 1 0.2 1"/>
+            </material>
+        </visual>
         <inertial>
             <origin xyz="0 0 0" rpy="0 0 0"/>
@@ -30,6 +47,6 @@
     </link>
     <joint name="rv_joint1" type="revolute">
-        <origin xyz="0 0.5 0" rpy="0 0 0"/>
-        <parent link="base_link"/>
+        <origin xyz="0 0.06 0" rpy="0 0 0"/>
+        <parent link="slider_link"/>
         <child link="sh_link"/>
         <axis xyz="0 0 1"/>
@@ -38,7 +55,7 @@
     <link name="sh_link">
         <visual>
-            <origin xyz="0 0.25 0" rpy="0 0 0"/>
+            <origin xyz="0 0.1525 0" rpy="0 0 0"/>
             <geometry>
-                <box size="0.1 0.5 0.1" />
+                <box size="0.032 0.185 0.01" />
             </geometry>
             <material name="green">
@@ -46,10 +63,4 @@
             </material>
         </visual>
-        <collision>
-            <origin xyz="0 0 0" rpy="0 0 0"/>
-            <geometry>
-                <box size="2.5 1.5 0.1" />
-            </geometry>
-        </collision>
         <inertial>
             <origin xyz="0 0 0" rpy="0 0 0"/>
@@ -58,9 +69,16 @@
         </inertial>
     </link>
-    <!-- <link name="base_link">
+    <joint name="rv_joint2" type="revolute">
+        <origin xyz="0 0.245 0" rpy="0 0 0"/>
+        <parent link="sh_link"/>
+        <child link="el_link"/>
+        <axis xyz="0 0 1"/>
+        <limit lower="-1.5708" upper="1.5708" velocity="0.5" effort="1000"/>
+    </joint>
+    <link name="el_link">
         <visual>
-            <origin xyz="0 0 0" rpy="0 0 0"/>
+            <origin xyz="0 0.0925 0" rpy="0 0 0"/>
             <geometry>
-                <box size="0.3 0.3 0.05" />
+                <box size="0.032 0.185 0.01" />
             </geometry>
             <material name="green">
@@ -68,10 +86,4 @@
             </material>
         </visual>
-        <collision>
-            <origin xyz="0 0 0" rpy="0 0 0"/>
-            <geometry>
-                <box size="2.5 1.5 0.1" />
-            </geometry>
-        </collision>
         <inertial>
             <origin xyz="0 0 0" rpy="0 0 0"/>
@@ -80,48 +92,3 @@
         </inertial>
     </link>
-    <joint name="fixed_joint1" type="fixed">
-        <origin xyz="0 0 0" rpy="0 0 0"/>
-        <parent link="base_link"/>
-        <child link="vert_support"/>
-    </joint>
-    <link name="vert_support">
-        <visual>
-            <origin xyz="0 0 0.25" rpy="0 0 0"/>
-            <geometry>
-                <box size="0.1 0.1 0.5" />
-            </geometry>
-            <material name="green">
-                <color rgba="0.2 1 0.2 1"/>
-            </material>
-        </visual>
-        <collision>
-            <origin xyz="0 0 0.05" rpy="0 0 0"/>
-            <geometry>
-                <box size="2.5 1.5 0.1" />
-            </geometry>
-        </collision>
-        <inertial>
-            <origin xyz="0 0 0.05" rpy="0 0 0"/>
-            <mass value="12" />
-            <inertia ixx="2.26" ixy="0.0" ixz="0.0" iyy="6.26" iyz="0.0" izz="8.5" />
-        </inertial>
-    </link>
-    <joint name="slider_joint" type="prismatic">
-        <origin xyz="0 0 0.05" rpy="0 0 0"/>
-        <parent link="vert_support"/>
-        <child link="slider"/>
-        <axis xyz="0 0 1"/>
-        <limit lower="0" upper="2" velocity="100" effort="100"/>
-    </joint>
-    <link name="slider">
-        <visual>
-            <origin xyz="0 0 0.05" rpy="0 0 0"/>
-            <geometry>
-                <box size="0.1 0.05 0.025" />
-            </geometry>
-            <material name="green">
-                <color rgba="0.2 1 0.2 1"/>
-            </material>
-        </visual>
-    </link> -->
 </robot>

Commit message: 1

File: v2scara/src/description/robot.urdf.xacro (robot description, xacro)
@@ -23,5 +23,5 @@
         </inertial>
     </link>
-    <joint name="slider_joint" type="prismatic">
+    <joint name="sl" type="prismatic">
         <origin xyz="0 0 0.445" rpy="0 0 0"/>
         <parent link="base_link"/>
@@ -46,10 +46,10 @@
         </inertial>
     </link>
-    <joint name="rv_joint1" type="revolute">
+    <joint name="sh" type="revolute">
         <origin xyz="0 0.06 0" rpy="0 0 0"/>
         <parent link="slider_link"/>
         <child link="sh_link"/>
         <axis xyz="0 0 1"/>
-        <limit lower="-1.5708" upper="1.5708" velocity="0.5" effort="1000"/>
+        <limit lower="1.5708" upper="-1.5708" velocity="0.5" effort="1000"/>
     </joint>
     <link name="sh_link">
@@ -69,10 +69,10 @@
         </inertial>
     </link>
-    <joint name="rv_joint2" type="revolute">
+    <joint name="el" type="revolute">
         <origin xyz="0 0.245 0" rpy="0 0 0"/>
         <parent link="sh_link"/>
         <child link="el_link"/>
         <axis xyz="0 0 1"/>
-        <limit lower="-1.5708" upper="1.5708" velocity="0.5" effort="1000"/>
+        <limit lower="1.5708" upper="-1.5708" velocity="0.5" effort="1000"/>
     </joint>
     <link name="el_link">
@@ -92,3 +92,26 @@
         </inertial>
     </link>
+    <joint name="cl" type="revolute">
+        <origin xyz="0 0 0" rpy="0 0 0"/>
+        <parent link="el_link"/>
+        <child link="cl_link"/>
+        <axis xyz="0 0 1"/>
+        <limit lower="1.5708" upper="-1.5708" velocity="0.5" effort="1000"/>
+    </joint>
+    <link name="cl_link">
+        <visual>
+            <origin xyz="0 0 0" rpy="0 0 0"/>
+            <geometry>
+                <box size="0.01 0.01 0.01" />
+            </geometry>
+            <material name="green">
+                <color rgba="0.2 1 0.2 1"/>
+            </material>
+        </visual>
+        <inertial>
+            <origin xyz="0 0 0" rpy="0 0 0"/>
+            <mass value="12" />
+            <inertia ixx="2.26" ixy="0.0" ixz="0.0" iyy="6.26" iyz="0.0" izz="8.5" />
+        </inertial>
+    </link>
 </robot>
